File: bitaxeUltraHex.kicad_pcb (KiCad board)
At the start: 4 copper layers, 136.3 x 79.7 mm, 291 parts, among them IC1 BM1397_mode1, IC2 BM1397_mode1, IC3 BM1397_mode0, IC4 BM1397_mode0, IC5 BM1397_mode1, IC6 BM1397_mode1, J1 Conn_01x01, J2 Conn_01x01, J3 Conn_01x04, J4 Conn_01x04, J5 TC2030-IDC, J6 Conn_01x04, J7 Conn_01x04, J8 Conn_01x05, Q1 NTMFS5C673NLT1G, Q2 CSD17577Q5A, Q3 NTMFS5C673NLT1G, Q4 CSD17577Q5A, SW1 GT-TC029B-H025-L1N, SW2 GT-TC029B-H025-L1N, U1 INA219AIDCNR, U10 EMC2101, U11 MCP1824T-1802E, U12 MCP1824T-0802E, U13 MCP1824T-1802E, U14 MCP1824T-0802E, U15 EMC2101, U16 SN74LVC1T45DBVR, U17 SN74LVC1T45DBVR, U18 SN74LVC1T45DBVR, U2 TPS40305, U3 uA7805, U4 RT9080-33GJ5, U5 DS4432U+, U6 ESP32-S3-WROOM-1, U7 MCP1824T-1802E, U8 MCP1824T-0802E, U9 EMC2101, X1 OT322525MJBA4SL, Y1 32.768kHz

Commit message: renamed hex to ultraHex
Parts:
- moved U3 203.3 mm to (134.0, 60.9)
- moved C153 175.7 mm to (153.1, 54.6)
- moved C154 175.7 mm to (153.1, 56.6)
- moved C155 175.7 mm to (153.1, 58.5)
- moved C156 175.7 mm to (153.1, 60.5)
- moved C157 175.7 mm to (153.1, 62.5)
- moved C158 175.7 mm to (153.1, 64.4)
- moved U16 175.7 mm to (149.2, 55.8)
- moved U17 175.7 mm to (149.2, 60.4)
- moved U18 175.7 mm to (149.2, 64.9)
- moved G*** 127.7 mm to (120.3, 133.7)
Changed lines of the file:
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@@
   )
   (footprint "Package_TO_SOT_SMD:TO-263-2" (layer "F.Cu")
-    (at -50.688 145.958 90)
+    (at 133.959 60.947 90)
     (descr "TO-263/D2PAK/DDPAK SMD package, http://www.infineon.com/cms/en/product/packages/PG-TO263/PG-TO263-3-1/")
     (tags "D2PAK DDPAK TO-263 D2PAK-3 TO-263-3 SOT-404")
@@
   )
   (footprint "LOGO" (layer "F.Cu")
-    (at 217.901 51.315)
+    (at 120.275659 133.711932)
     (attr board_only exclude_from_pos_files exclude_from_bom)
     (fp_text reference "G***" (at -0.408 5.806) (layer "F.SilkS") hide
@@
   )
   (footprint "Capacitor_SMD:C_0402_1005Metric" (layer "F.Cu")
-    (at -9.282 129.509)
+    (at 153.08 62.471)
     (descr "Capacitor SMD 0402 (1005 Metric), square (rectangular) end terminal, IPC_7351 nominal, (Body size source: IPC-SM-782 page 76, https://www.pcb-3d.com/wordpress/wp-content/uploads/ipc-sm-782a_amendment_1_and_2.pdf), generated with kicad-footprint-generator")
     (tags "capacitor")
@@
   )
   (footprint "lcsc:SOT-23-6_L2.9-W1.6-P0.95-LS2.8-BR" (layer "F.Cu")
-    (at -13.117 131.979)
+    (at 149.245 64.941)
     (property "JLC Part" "Extended Part")
     (property "LCSC Part" "C7843")
@@
   )
   (footprint "Capacitor_SMD:C_0402_1005Metric" (layer "F.Cu")
-    (at -9.282 121.629)
+    (at 153.08 54.591)
     (descr "Capacitor SMD 0402 (1005 Metric), square (rectangular) end terminal, IPC_7351 nominal, (Body size source: IPC-SM-782 page 76, https://www.pcb-3d.com/wordpress/wp-content/uploads/ipc-sm-782a_amendment_1_and_2.pdf), generated with kicad-footprint-generator")
     (tags "capacitor")
@@
   )
   (footprint "Capacitor_SMD:C_0402_1005Metric" (layer "F.Cu")
-    (at -9.282 125.569)
+    (at 153.08 58.531)
     (descr "Capacitor SMD 0402 (1005 Metric), square (rectangular) end terminal, IPC_7351 nominal, (Body size source: IPC-SM-782 page 76, https://www.pcb-3d.com/wordpress/wp-content/uploads/ipc-sm-782a_amendment_1_and_2.pdf), generated with kicad-footprint-generator")
     (tags "capacitor")
@@
   )
   (footprint "lcsc:SOT-23-6_L2.9-W1.6-P0.95-LS2.8-BR" (layer "F.Cu")
-    (at -13.117 127.399)
+    (at 149.245 60.361)
     (property "JLC Part" "Extended Part")
     (property "LCSC Part" "C7843")
@@
   )
   (footprint "Capacitor_SMD:C_0402_1005Metric" (layer "F.Cu")
-    (at -9.282 123.599)
+    (at 153.08 56.561)
     (descr "Capacitor SMD 0402 (1005 Metric), square (rectangular) end terminal, IPC_7351 nominal, (Body size source: IPC-SM-782 page 76, https://www.pcb-3d.com/wordpress/wp-content/uploads/ipc-sm-782a_amendment_1_and_2.pdf), generated with kicad-footprint-generator")
     (tags "capacitor")
@@
   )
   (footprint "Capacitor_SMD:C_0402_1005Metric" (layer "F.Cu")
-    (at -9.282 131.479)
+    (at 153.08 64.441)
     (descr "Capacitor SMD 0402 (1005 Metric), square (rectangular) end terminal, IPC_7351 nominal, (Body size source: IPC-SM-782 page 76, https://www.pcb-3d.com/wordpress/wp-content/uploads/ipc-sm-782a_amendment_1_and_2.pdf), generated with kicad-footprint-generator")
     (tags "capacitor")
@@
   )
   (footprint "lcsc:SOT-23-6_L2.9-W1.6-P0.95-LS2.8-BR" (layer "F.Cu")
-    (at -13.117 122.819)
+    (at 149.245 55.781)
     (property "JLC Part" "Extended Part")
     (property "LCSC Part" "C7843")
@@
   )
   (footprint "Capacitor_SMD:C_0402_1005Metric" (layer "F.Cu")
-    (at -9.282 127.539)
+    (at 153.08 60.501)
     (descr "Capacitor SMD 0402 (1005 Metric), square (rectangular) end terminal, IPC_7351 nominal, (Body size source: IPC-SM-782 page 76, https://www.pcb-3d.com/wordpress/wp-content/uploads/ipc-sm-782a_amendment_1_and_2.pdf), generated with kicad-footprint-generator")
     (tags "capacitor")

Commit message: moved all custom symbols and footprints to the bitaxe library
Parts:
- removed C129, C130, C131, C132, C133, C134, C135, C136, C138, C140, C141, C142, C144, C145, C146, C147, C148: 587-5514-1-ND, Capacitor_SMD:C_0402_1005Metric
- removed C137, C139, C150, C152, C153, C154, C155, C156, C157, C158: 311-3342-1-ND, Capacitor_SMD:C_0402_1005Metric
- removed C143: 330uF, Capacitor_Tantalum_SMD:CP_EIA-7343-31_Kemet-D_Pad2.25x2.55mm_HandSolder
- removed C149: 470pF, Capacitor_SMD:C_0402_1005Metric
- removed C151: 220uF, Capacitor_SMD:CP_Elec_6.3x7.7
- removed IC1, IC2, IC5, IC6: BM1397_mode1, bitaxe:BM1397
- removed IC3, IC4: BM1397_mode0, bitaxe:BM1397
- removed J7: Conn_01x04, bitaxe:470531000
- removed J8: Conn_01x05, Connector_PinHeader_2.54mm:PinHeader_1x05_P2.54mm_Vertical
- removed TP20, TP21, TP22, TP23, TP24, TP25, TP26, TP27, TP28, TP29, TP30, TP31, TP32, TP33, TP34: TestPoint, TestPoint:TestPoint_Pad_D1.5mm
- removed X1: OT322525MJBA4SL, lcsc:OSC-SMD_4P-L3.2-W2.5-BL
- added R43: 33, Resistor_SMD:R_0402_1005Metric, F.Cu at (28.9, 115.5)
- added R44: 33, Resistor_SMD:R_0402_1005Metric, F.Cu at (28.9, 117.5)
- added R52: 6.8k, Resistor_SMD:R_0402_1005Metric, F.Cu at (23.7, 95.0)
- added R53: 6.8k, Resistor_SMD:R_0402_1005Metric, F.Cu at (23.7, 97.0)
- added R54: 1, Resistor_SMD:R_2512_6332Metric, F.Cu at (35.4, 96.4)
- added R55: 33, Resistor_SMD:R_0402_1005Metric, F.Cu at (23.7, 99.0)
- added R56: 1, Resistor_SMD:R_2512_6332Metric, F.Cu at (35.4, 101.3)
- added R57: 33, Resistor_SMD:R_0402_1005Metric, F.Cu at (23.7, 101.0)
- added R58: 33, Resistor_SMD:R_0402_1005Metric, F.Cu at (23.7, 103.0)
- added R59: 33, Resistor_SMD:R_0402_1005Metric, F.Cu at (26.6, 95.0)
- added R60: 33, Resistor_SMD:R_0402_1005Metric, F.Cu at (26.6, 97.0)
- added R61: 33, Resistor_SMD:R_0402_1005Metric, F.Cu at (26.6, 99.0)
- added R62: 33, Resistor_SMD:R_0402_1005Metric, F.Cu at (26.6, 101.0)
- added R63: 6.8k, Resistor_SMD:R_0402_1005Metric, F.Cu at (26.6, 103.0)
- added R64: 33, Resistor_SMD:R_0402_1005Metric, F.Cu at (29.6, 95.0)
- added R65: 33, Resistor_SMD:R_0402_1005Metric, F.Cu at (29.6, 97.0)
- added R66: 33, Resistor_SMD:R_0402_1005Metric, F.Cu at (29.6, 99.0)
- added TP15: TestPoint, TestPoint:TestPoint_Pad_D1.5mm, F.Cu at (39.8, 87.2)
- added U19: MCP1824T-1202E, Package_TO_SOT_SMD:SOT-23-5, F.Cu at (24.9, 116.7)
- added U20: MCP1824T-0802E, Package_TO_SOT_SMD:SOT-23-5, F.Cu at (24.9, 121.2)
- added U21: BM1366_mode1, bitaxe:BM1366, F.Cu at (26.3, 110.5)
- added U22: BM1366_mode1, bitaxe:BM1366, F.Cu at (34.2, 110.5)
- added U23: MCP1824T-1202E, Package_TO_SOT_SMD:SOT-23-5, F.Cu at (42.3, 96.2)
- added U24: MCP1824T-0802E, Package_TO_SOT_SMD:SOT-23-5, F.Cu at (42.3, 100.7)
- added U25: BM1366_mode1, bitaxe:BM1366, F.Cu at (26.3, 90.0)
- added U26: BM1366_mode1, bitaxe:BM1366, F.Cu at (34.2, 90.0)
- C10: value 0.33uF -> 3.3nF
- C100, C102, C103, C104, C108, C109, C110, C111, C112, C113, C114, C115, C119, C121, C122, C125, C127, C128, C35, C38, C43, C44, C45, C46, C47, C48, C49, C50, C51, C52, C54, C56, C57, C58, C60, C75, C76, C77, C81, C84, C87, C89, C90, C91, C92, C93, C94, C95, C96, C97, C98: value 587-5514-1-ND -> 1uF
- C101, C116, C117, C118, C120, C32, C33, C34, C36, C53, C55, C68, C71, C72, C78, C79, C82, C99: value 311-3342-1-ND -> 1uF
- C105, C126, C42, C59: value 330uF -> 1uF; footprint Capacitor_Tantalum_SMD:CP_EIA-7343-31_Kemet-D_Pad2.25x2.55mm_HandSolder -> Capacitor_SMD:C_0402_1005Metric
- C106, C107, C37, C41, C73, C74, C83: value 587-5514-1-ND -> 0.1uF
- C11, C40: value 1uF -> 0.1uF
- C12: value 0.1uF -> 1uF
- C13: value 4.7uF -> 1uF; footprint Capacitor_SMD:C_0805_2012Metric -> Capacitor_SMD:C_0402_1005Metric
- C15: value 1uF -> 4.7uF; footprint Capacitor_SMD:C_0402_1005Metric -> Capacitor_SMD:C_0805_2012Metric
- C21: value 1uF -> 10uF; footprint Capacitor_SMD:C_0402_1005Metric -> Capacitor_SMD:C_0805_2012Metric
- C22: value 10uF -> 1uF; footprint Capacitor_SMD:C_0805_2012Metric -> Capacitor_SMD:C_0402_1005Metric
- C23: value 6.8pF -> 0.1uF
- C24: value 0.1uF -> 311-3342-1-ND
- C25: value 6.8pF -> 311-3342-1-ND
- C27, C28, C29, C61, C62, C63: value 587-5514-1-ND -> 311-3342-1-ND
- C3: value ~ -> 0.33uF
- C30, C31: value 587-5514-1-ND -> 6.8pF
- C4: value 22uF -> ~; footprint Capacitor_SMD:C_2220_5650Metric -> Capacitor_SMD:C_0402_1005Metric
- C5: footprint Capacitor_SMD:C_0805_2012Metric -> Capacitor_SMD:C_0402_1005Metric
- C6: value 3.3nF -> 22uF; footprint Capacitor_SMD:C_0402_1005Metric -> Capacitor_SMD:C_2220_5650Metric
- C64: value 587-5514-1-ND -> 220uF; footprint Capacitor_SMD:C_0402_1005Metric -> Capacitor_SMD:CP_Elec_6.3x7.7
- C65: value 470pF -> 220uF; footprint Capacitor_SMD:C_0402_1005Metric -> Capacitor_SMD:CP_Elec_6.3x7.7
- C66: value 470pF -> 311-3342-1-ND
- C69, C70: value 220uF -> 1uF; footprint Capacitor_SMD:CP_Elec_6.3x7.7 -> Capacitor_SMD:C_0402_1005Metric
- C8: value 5.6nF -> 1uF
- C80: value 311-3342-1-ND -> 0.1uF
- C9: value 1uF -> 5.6nF; footprint Capacitor_SMD:C_0402_1005Metric -> Capacitor_SMD:C_0805_2012Metric
- D1: footprint lcsc:SMA_L4.3-W2.6-LS5.2-RD -> bitaxe:SMA_L4.3-W2.6-LS5.2-RD
- J1, J2: footprint TPS40305_supply:63862-1 -> bitaxe:63862-1
- J3: footprint bitaxe:470531000 -> Connector_PinHeader_2.54mm:PinHeader_1x04_P2.54mm_Vertical
- J4: value Conn_01x04 -> TC2030-IDC; footprint Connector_PinHeader_2.54mm:PinHeader_1x04_P2.54mm_Vertical -> bitaxe:Tag-Connect_TC2030-IDC-NL_2x03_P1.27mm_Vertical
- J5: value TC2030-IDC -> Conn_01x04; footprint Connector:Tag-Connect_TC2030-IDC-NL_2x03_P1.27mm_Vertical -> bitaxe:470531000
- Q1: footprint bitaxe:NTMFS5C673NLT1G -> bitaxe:CSD17311Q5
- R10: value DNP -> 1.54k
- R11: value 10k -> 80k
- R12: value 1.54k -> DNP
- R16, R32: value 0 -> 10k
- R17, R18, R37, R47: value 0 -> 6.8k
- R19, R20: value 1 -> 33; footprint Resistor_SMD:R_2512_6332Metric -> Resistor_SMD:R_0402_1005Metric
- R21, R22, R23, R39, R41, R42, R45, R46: value 0 -> 33
- R24, R25: value 100 -> 1; footprint Resistor_SMD:R_0402_1005Metric -> Resistor_SMD:R_2512_6332Metric
- R26, R27, R48, R49: value 100 -> 33
- R28: value 10k -> 6.8k
- R29, R50: value 10k -> 33
- R30, R31: value 5.6k -> 33
- R33, R34: value 0 -> 5.6k
- R35: value 1 -> 10k; footprint Resistor_SMD:R_2512_6332Metric -> Resistor_SMD:R_0402_1005Metric
- R36: value 1 -> 6.8k; footprint Resistor_SMD:R_2512_6332Metric -> Resistor_SMD:R_0402_1005Metric
- R38, R40: value 0 -> 1; footprint Resistor_SMD:R_0402_1005Metric -> Resistor_SMD:R_2512_6332Metric
- R5: value 10k -> 100k
- R51: value 5.6k -> 10k
- R6: value 100k -> 6.49k
- R7: value 6.49k -> 10k
- R8: value 80k -> 487
- R9: value 487 -> 10k
- U1: value INA219AIDCNR -> uA7805; footprint lcsc:SOT-23-8_L3.0-W1.7-P0.65-LS2.8-BR -> Package_TO_SOT_SMD:TO-263-2
- U10: value EMC2101 -> 25MHz; footprint Package_SO:TSSOP-8_3x3mm_P0.65mm -> bitaxe:O 25,0-JO32-B-1V3-1-T1-LF
- U11: value MCP1824T-1802E -> BM1366_mode1; footprint Package_TO_SOT_SMD:SOT-23-5 -> bitaxe:BM1366
- U12: value MCP1824T-0802E -> MCP1824T-1202E
- U13: value MCP1824T-1802E -> MCP1824T-0802E
- U14: value MCP1824T-0802E -> BM1366_mode1; footprint Package_TO_SOT_SMD:SOT-23-5 -> bitaxe:BM1366
- U15: value EMC2101 -> TMP1075; footprint Package_SO:TSSOP-8_3x3mm_P0.65mm -> bitaxe:SOT5X3-6_DRL_TEX
- U16: value SN74LVC1T45DBVR -> TMP1075; footprint lcsc:SOT-23-6_L2.9-W1.6-P0.95-LS2.8-BR -> bitaxe:SOT5X3-6_DRL_TEX
- U17: value SN74LVC1T45DBVR -> EMC2302; footprint lcsc:SOT-23-6_L2.9-W1.6-P0.95-LS2.8-BR -> Package_SO:MSOP-10_3x3mm_P0.5mm
- U18: value SN74LVC1T45DBVR -> EMC2101; footprint lcsc:SOT-23-6_L2.9-W1.6-P0.95-LS2.8-BR -> Package_SO:TSSOP-8_3x3mm_P0.65mm
- U2: value TPS40305 -> RT9080-33GJ5; footprint TPS40305_supply:TPS40305 -> bitaxe:RT9080-33GJ5
- U3: value uA7805 -> INA219AIDCNR; footprint Package_TO_SOT_SMD:TO-263-2 -> Package_TO_SOT_SMD:SOT-23-8
- U4: value RT9080-33GJ5 -> TPS40305; footprint bitaxe:RT9080-33GJ5 -> bitaxe:TPS40305
- U6: value ESP32-S3-WROOM-1 -> SN74LVC1T45DBVR; footprint Espressif:ESP32-S3-WROOM-1 -> lcsc:SOT-23-6_L2.9-W1.6-P0.95-LS2.8-BR
- U7: value MCP1824T-1802E -> SN74LVC1T45DBVR; footprint Package_TO_SOT_SMD:SOT-23-5 -> lcsc:SOT-23-6_L2.9-W1.6-P0.95-LS2.8-BR
- U8: value MCP1824T-0802E -> SN74LVC1T45DBVR; footprint Package_TO_SOT_SMD:SOT-23-5 -> lcsc:SOT-23-6_L2.9-W1.6-P0.95-LS2.8-BR
- U9: value EMC2101 -> ESP32-S3-WROOM-1; footprint Package_SO:TSSOP-8_3x3mm_P0.65mm -> bitaxe:ESP32-S3-WROOM-1
- USB1: footprint lcsc:MICRO-USB-SMD_U254-051T-4BHJ25-F2S -> bitaxe:MICRO-USB-SMD_U254-051T-4BHJ25-F2S
- moved U1 25.4 mm to (-5.55, 104.2)
Connections:
- C10 pad 1: /Power/VIN_M -> Net-(U4-SS)
- C100 pad 2: /BM1397-1/GND1 -> Net-(C100-Pad2)
- C101 pad 1: /BM1397-1/GND1 -> Net-(C101-Pad1)
- C101 pad 2: /BM1397-3/VDD3 -> Net-(U25-VDD3_0)
- C102 pad 1: /BM1397-1/GND1 -> Net-(U25-MODEO)
- C102 pad 2: /BM1397-3/VDD3 -> /BM1366-3/0V8
- C103 pad 1: /BM1397-1/GND1 -> Net-(U25-VDD3_0)
- C103 pad 2: /BM1397-3/VDD3 -> Net-(U25-VDD2_0)
- C104 pad 1: /BM1397-1/GND1 -> /BM1366-3/1V2
- C104 pad 2: Net-(IC4-VDD3_1) -> GND
- C105 pad 1: /BM1397-1/GND1 -> Net-(U25-VDD2_0)
- C105 pad 2: /BM1397-3/VDD3 -> Net-(U25-VDD1_0)
- C106 pad 1: Net-(IC4-VDD3_1) -> /5V
- C106 pad 2: Net-(IC4-VDD2_1) -> GND
- C107 pad 1: /BM1398-2/1V8 -> /5V
- C107 pad 2: /BM1397-3/VDD3 -> GND
- C108 pad 1: /BM1398-2/0V8 -> Net-(U25-VDD1_0)
- C108 pad 2: /BM1397-3/VDD3 -> /BM1366-2/GND
- C109 pad 1: Net-(IC4-VDD2_1) -> /BM1366-3/1V2
- C109 pad 2: Net-(IC4-VDD1_1) -> GND
- C110 pad 1: Net-(IC4-VDD1_1) -> /BM1366-3/0V8
- C110 pad 2: /BM1397-3/VDD3 -> GND
- C111 pad 1: GND -> /BM1366-3/1V2
- C111 pad 2: Net-(IC5-VDD1_0) -> GND
- C112 pad 1: Net-(IC5-VDD1_0) -> /BM1366-2/GND
- C112 pad 2: Net-(IC5-VDD2_0) -> Net-(U25-VDD1_1)
- C113 pad 1: /BM1397-3/0V8 -> Net-(U25-VDD1_1)
- C113 pad 2: GND -> Net-(U25-VDD2_1)
- C114 pad 1: /BM1397-3/1V8 -> Net-(U25-MODE_1)
- C114 pad 2: GND -> /BM1366-3/0V8
- C115 pad 1: Net-(IC5-VDD2_0) -> Net-(U25-VDD2_1)
- C115 pad 2: Net-(IC5-VDD3_0) -> Net-(U25-VDD3_1)
- C116 pad 1: /BM1397-3/VDD3 -> Net-(U25-VDD3_1)
- C116 pad 2: GND -> Net-(C116-Pad2)
- C117 pad 1: /5V -> Net-(C116-Pad2)
- C117 pad 2: GND -> Net-(U25-VDD3_1)
- C118 pad 1: /5V -> Net-(U25-VDD3_1)
- C118 pad 2: GND -> Net-(U25-VDD2_1)
- C119 pad 1: Net-(IC5-VDD3_0) -> Net-(U25-MODE_1)
- C119 pad 2: /BM1397-3/VDD3 -> /BM1366-3/0V8
- C12 pad 1: Net-(U2-BOOT) -> /3V3
- C12 pad 2: /Power/SW -> GND
- C120 pad 1: /BM1397-3/VDD3 -> Net-(U25-VDD2_1)
- C120 pad 2: GND -> Net-(U25-VDD1_1)
- C121 pad 1: /BM1397-3/VDD3 -> /BM1366-3/1V2
- C122 pad 1: /BM1397-3/VDD3 -> Net-(U25-VDD1_1)
- C122 pad 2: GND -> /BM1366-2/GND
- C123 pad 1: /BM1397-3/1V8 -> /BM1366-2/GND
- C123 pad 2: GND -> Net-(U26-VDD1_1)
- C124 pad 1: /BM1397-3/0V8 -> Net-(U26-VDD1_1)
- C124 pad 2: GND -> Net-(U26-VDD2_1)
- C125 pad 1: /BM1397-3/VDD3 -> /BM1366-3/1V2
- C125 pad 2: Net-(IC5-VDD3_1) -> GND
- C126 pad 1: /BM1397-3/VDD3 -> Net-(U26-VDD2_1)
- C126 pad 2: GND -> Net-(U26-VDD3_1)
- C127 pad 1: Net-(IC5-VDD3_1) -> /BM1366-3/0V8
- C128 pad 1: /BM1397-3/1V8 -> Net-(U26-VDD3_1)
- C128 pad 2: GND -> Net-(C128-Pad2)
- C13 pad 1: Net-(U2-BP) -> /3V3
- C14 pad 1: /5V -> Net-(U4-BOOT)
- C14 pad 2: GND -> /Power/SW
- C15 pad 1: /3V3 -> Net-(U4-BP)
- C21 pad 1: /ESP32/EN -> /3V3
- C22 pad 1: /3V3 -> /ESP32/EN
- C23 pad 1: /ESP32/XIN32 -> /3V3
- C24 pad 1: /3V3 -> /1V8
- C25 pad 1: /ESP32/XOUT32 -> /1V8
- C26 pad 1: /BM1397-1/GND1 -> /1V8
- C26 pad 2: /1V8 -> GND
- C27 pad 1: /BM1397-1/GND1 -> /3V3
- C27 pad 2: Net-(IC1-VDD1_0) -> GND
- C28 pad 1: Net-(IC1-VDD1_0) -> /3V3
- C28 pad 2: Net-(IC1-VDD2_0) -> GND
- C29 pad 1: /BM1397-1/0V8 -> /3V3
- C29 pad 2: /BM1397-1/GND1 -> GND
- C3 pad 1: Net-(U1-IN+) -> /Power/VIN_M
- C3 pad 2: Net-(U1-IN-) -> GND
- C30 pad 1: /1V8 -> /ESP32/XIN32
- C30 pad 2: /BM1397-1/GND1 -> GND
- C31 pad 1: Net-(IC1-VDD2_0) -> /ESP32/XOUT32
- C31 pad 2: Net-(IC1-VDD3_0) -> GND
- C32 pad 1: /5V -> Net-(C32-Pad1)
- C32 pad 2: /BM1397-1/GND1 -> Net-(U11-VDD3_0)
- C33 pad 1: /5V -> Net-(U11-MODEO)
- C33 pad 2: /BM1397-1/GND1 -> /BM1366-1/0V8
- C34 pad 1: /VDD -> Net-(U11-VDD3_0)
- C34 pad 2: /BM1397-1/GND1 -> Net-(U11-VDD2_0)
- C35 pad 1: Net-(IC1-VDD3_0) -> /BM1366-1/1V2
- C35 pad 2: /VDD -> /BM1366-1/GND
- C36 pad 1: /VDD -> Net-(U11-VDD2_0)
- C36 pad 2: /BM1397-1/GND1 -> Net-(U11-VDD1_0)
- C37 pad 1: /VDD -> /BM1366-1/GND
- C37 pad 2: /BM1397-1/GND1 -> /BM1366-1/1V2
- C38 pad 1: /VDD -> Net-(U11-VDD1_0)
- C38 pad 2: /BM1397-1/GND1 -> /VDD
- C39 pad 1: /1V8 -> /BM1366-1/1V2
- C39 pad 2: /BM1397-1/GND1 -> /BM1366-1/GND
- C4 pad 1: /Power/VIN_M -> Net-(U3-IN+)
- C4 pad 2: GND -> Net-(U3-IN-)
- C40 pad 1: /BM1397-1/0V8 -> /5V
- C40 pad 2: /BM1397-1/GND1 -> /BM1366-1/GND
- C41 pad 1: /VDD -> /5V
- C41 pad 2: Net-(IC1-VDD3_1) -> /BM1366-1/GND
- C42 pad 2: /BM1397-1/GND1 -> Net-(U11-VDD1_1)
- C43 pad 1: Net-(IC1-VDD3_1) -> Net-(U11-VDD1_1)
- C43 pad 2: Net-(IC1-VDD2_1) -> Net-(U11-VDD2_1)
- C44 pad 1: /1V8 -> Net-(U11-MODE_1)
- C44 pad 2: /BM1397-1/GND1 -> /BM1366-1/0V8
- C45 pad 1: /BM1397-1/0V8 -> Net-(U11-VDD2_1)
- C45 pad 2: /BM1397-1/GND1 -> Net-(U11-VDD3_1)
- C46 pad 1: Net-(IC1-VDD2_1) -> /BM1366-1/1V2
- C46 pad 2: Net-(IC1-VDD1_1) -> /BM1366-1/GND
- C47 pad 1: Net-(IC1-VDD1_1) -> /BM1366-1/0V8
- C47 pad 2: /BM1397-1/GND1 -> /BM1366-1/GND
- C48 pad 1: /BM1397-1/GND1 -> Net-(U11-VDD3_1)
- C48 pad 2: Net-(IC2-VDD1_0) -> Net-(C48-Pad2)
- C49 pad 1: Net-(IC2-VDD1_0) -> Net-(C48-Pad2)
- C49 pad 2: Net-(IC2-VDD2_0) -> Net-(U11-VDD3_1)
- C5 pad 1: /Power/VIN_M -> /5V
- C50 pad 1: /BM1397-1/0V8 -> Net-(U11-VDD3_1)
- C50 pad 2: /BM1397-1/GND1 -> Net-(U11-VDD2_1)
- C51 pad 1: /1V8 -> Net-(U11-MODE_1)
- C51 pad 2: /BM1397-1/GND1 -> /BM1366-1/0V8
- C52 pad 1: Net-(IC2-VDD2_0) -> Net-(U11-VDD2_1)
- C52 pad 2: Net-(IC2-VDD3_0) -> Net-(U11-VDD1_1)
- C53 pad 1: /VDD -> /BM1366-1/1V2
- C53 pad 2: /BM1397-1/GND1 -> /BM1366-1/GND
- C54 pad 1: Net-(IC2-VDD3_0) -> Net-(U11-VDD1_1)
- C55 pad 2: /BM1397-1/GND1 -> Net-(U14-VDD1_1)
- C56 pad 1: /VDD -> Net-(U14-VDD1_1)
- C56 pad 2: /BM1397-1/GND1 -> Net-(U14-VDD2_1)
- C57 pad 1: /VDD -> /BM1366-1/1V2
- C57 pad 2: /BM1397-1/GND1 -> /BM1366-1/GND
- C58 pad 1: /VDD -> Net-(U14-VDD2_1)
- C58 pad 2: Net-(IC2-VDD3_1) -> Net-(U14-VDD3_1)
- C59 pad 1: /VDD -> /BM1366-1/0V8
- C59 pad 2: /BM1397-1/GND1 -> Net-(U14-MODE_1)
- C6 pad 1: Net-(U2-SS) -> /Power/VIN_M
- C60 pad 1: Net-(IC2-VDD3_1) -> Net-(U14-VDD3_1)
- C60 pad 2: Net-(IC2-VDD2_1) -> Net-(C60-Pad2)
- C61 pad 1: /1V8 -> /3V3
- C61 pad 2: /BM1397-1/GND1 -> GND
- C62 pad 1: /BM1397-1/0V8 -> unconnected-(C62-Pad1)
- C62 pad 2: /BM1397-1/GND1 -> unconnected-(C62-Pad2)
- C63 pad 1: Net-(IC2-VDD2_1) -> unconnected-(C63-Pad1)
- C63 pad 2: Net-(IC2-VDD1_1) -> unconnected-(C63-Pad2)
- C64 pad 1: Net-(IC2-VDD1_1) -> /5V
- C64 pad 2: /BM1397-1/GND1 -> GND
- C65 pad 1: Net-(U9-DP) -> /5V
- C65 pad 2: Net-(U9-DN) -> GND
- C66 pad 1: Net-(U10-DP) -> /5V
- C66 pad 2: Net-(U10-DN) -> GND
- C67 pad 1: /3V3 -> /5V
- C68 pad 1: /3V3 -> Net-(C68-Pad1)
- C68 pad 2: GND -> Net-(U21-VDD3_0)
- C69 pad 1: /5V -> Net-(U21-MODEO)
- C69 pad 2: GND -> /BM1366-2/0V8
- C7 pad 1: Net-(U2-COMP) -> Net-(U4-COMP)
- C70 pad 1: /5V -> Net-(U21-VDD3_0)
- C70 pad 2: GND -> Net-(U21-VDD2_0)
- C71 pad 1: /5V -> /BM1366-2/1V2
- C71 pad 2: GND -> /BM1366-2/GND
- C72 pad 1: /5V -> Net-(U21-VDD2_0)
- C72 pad 2: GND -> Net-(U21-VDD1_0)
- C73 pad 1: /BM1397-3/VDD3 -> /5V
- C73 pad 2: Net-(IC3-VDD1_0) -> /BM1366-2/GND
- C74 pad 1: Net-(IC3-VDD1_0) -> /5V
- C74 pad 2: Net-(IC3-VDD2_0) -> /BM1366-2/GND
- C75 pad 1: /BM1398-2/0V8 -> Net-(U21-VDD1_0)
- C75 pad 2: /BM1397-3/VDD3 -> /BM1366-1/GND
- C76 pad 1: /BM1398-2/1V8 -> /BM1366-2/1V2
- C76 pad 2: /BM1397-3/VDD3 -> /BM1366-2/GND
- C77 pad 1: Net-(IC3-VDD2_0) -> /BM1366-2/0V8
- C77 pad 2: Net-(IC3-VDD3_0) -> /BM1366-2/GND
- C78 pad 1: /BM1397-1/GND1 -> /BM1366-2/1V2
- C78 pad 2: /BM1397-3/VDD3 -> /BM1366-2/GND
- C79 pad 1: /5V -> /BM1366-1/GND
- C79 pad 2: /BM1397-3/VDD3 -> Net-(U21-VDD1_1)
- C8 pad 1: Net-(U2-COMP) -> /Power/VIN_M
- C8 pad 2: Net-(C8-Pad2) -> GND
- C80 pad 1: /5V -> /BM1366-1/GND
- C80 pad 2: /BM1397-3/VDD3 -> /BM1366-2/GND
- C81 pad 1: Net-(IC3-VDD3_0) -> Net-(U21-VDD1_1)
- C81 pad 2: /BM1397-1/GND1 -> Net-(U21-VDD2_1)
- C82 pad 1: /BM1397-1/GND1 -> Net-(U21-MODE_1)
- C82 pad 2: /BM1397-3/VDD3 -> /BM1366-2/0V8
- C83 pad 1: /BM1397-1/GND1 -> /BM1366-1/GND
- C83 pad 2: /BM1397-3/VDD3 -> /BM1366-2/GND
- C84 pad 1: /BM1397-1/GND1 -> Net-(U21-VDD2_1)
- C84 pad 2: /BM1397-3/VDD3 -> Net-(U21-VDD3_1)
- C85 pad 1: /BM1398-2/1V8 -> /BM1366-1/GND
- C85 pad 2: /BM1397-3/VDD3 -> /BM1366-2/GND
- C86 pad 1: /BM1398-2/0V8 -> Net-(U21-VDD3_1)
- C86 pad 2: /BM1397-3/VDD3 -> Net-(C86-Pad2)
- C87 pad 1: /BM1397-1/GND1 -> /BM1366-1/GND
- C87 pad 2: Net-(IC3-VDD3_1) -> /BM1366-2/GND
- C88 pad 1: /BM1397-1/GND1 -> /BM1366-1/GND
- C88 pad 2: /BM1397-3/VDD3 -> /BM1366-2/GND
- C89 pad 1: Net-(IC3-VDD3_1) -> Net-(C86-Pad2)
- C89 pad 2: Net-(IC3-VDD2_1) -> Net-(U21-VDD3_1)
- C9 pad 1: /3V3 -> Net-(U4-COMP)
- C9 pad 2: GND -> Net-(C9-Pad2)
- C90 pad 1: /BM1398-2/1V8 -> Net-(U21-VDD3_1)
- C90 pad 2: /BM1397-3/VDD3 -> Net-(U21-VDD2_1)
- C91 pad 1: /BM1398-2/0V8 -> Net-(U21-MODE_1)
- C91 pad 2: /BM1397-3/VDD3 -> /BM1366-2/0V8
- C92 pad 1: Net-(IC3-VDD2_1) -> Net-(U21-VDD2_1)
- C92 pad 2: Net-(IC3-VDD1_1) -> Net-(U21-VDD1_1)
- C93 pad 1: Net-(IC3-VDD1_1) -> /BM1366-2/1V2
- C93 pad 2: /BM1397-3/VDD3 -> /BM1366-2/GND
- C94 pad 1: /BM1397-3/VDD3 -> Net-(U21-VDD1_1)
- C94 pad 2: Net-(IC4-VDD1_0) -> /BM1366-1/GND
- C95 pad 1: Net-(IC4-VDD1_0) -> /BM1366-1/GND
- C95 pad 2: Net-(IC4-VDD2_0) -> Net-(U22-VDD1_1)
- C96 pad 1: /BM1398-2/0V8 -> Net-(U22-VDD1_1)
- C96 pad 2: /BM1397-3/VDD3 -> Net-(U22-VDD2_1)
- C97 pad 1: /BM1398-2/1V8 -> /BM1366-2/1V2
- C97 pad 2: /BM1397-3/VDD3 -> /BM1366-2/GND
- C98 pad 1: Net-(IC4-VDD2_0) -> Net-(U22-VDD2_1)
- C99 pad 1: /BM1397-1/GND1 -> /BM1366-2/0V8
- C99 pad 2: /BM1397-3/VDD3 -> Net-(U22-MODE_1)
- J3 pad 2: /5V -> /3V3
- J3 pad 3: /Fan/FAN_TACH3 -> /SCL
- J3 pad 4: /Fan/FAN_PWM3 -> /SDA
- J4 pad 1: GND -> /ESP32/EN
- J4 pad 3: /SCL -> /ESP32/P_TX
- J4 pad 4: /SDA -> GND
- J5 pad 1: /ESP32/EN -> GND
- J5 pad 2: /3V3 -> /5V
- J5 pad 3: /ESP32/P_TX -> /Fan/FAN1_TACH
- J5 pad 4: GND -> /Fan/FAN1_PWM
- J6 pad 3: /Fan/FAN_TACH1 -> /Fan/FAN2_TACH
- J6 pad 4: /Fan/FAN_PWM1 -> /Fan/FAN2_PWM
- R10 pad 1: Net-(U5-FS1) -> /Power/OUT0
- R11 pad 1: /VDD -> Net-(U5-FS0)
- R11 pad 2: /Power/OUT0 -> GND
- R12 pad 1: /Power/OUT0 -> Net-(U5-FS1)
- R16 pad 1: /BM1397-1/GND1 -> /BM1366-1/GND
- R16 pad 2: Net-(IC1-ADDR0) -> Net-(U11-BI)
- R17 pad 1: /BM1397-1/GND1 -> Net-(U11-NC)
- R17 pad 2: Net-(IC1-ADDR1) -> Net-(U11-MODE_1)
- R18 pad 1: /BM1397-1/GND1 -> Net-(C48-Pad2)
- R18 pad 2: Net-(IC1-ADDR2) -> Net-(U11-NRSTO)
- R19 pad 1: /VDD -> Net-(U11-RI)
- R19 pad 2: /BM1397-1/GND1 -> Net-(U14-RO)
- R2 pad 2: Net-(U1-IN+) -> Net-(U3-IN+)
- R20 pad 1: /VDD -> Net-(U11-BO)
- R20 pad 2: /BM1397-1/GND1 -> Net-(U14-BI)
- R21 pad 1: /BM1397-1/GND1 -> Net-(U11-CLKO)
- R21 pad 2: Net-(IC2-ADDR0) -> Net-(U14-CLKI)
- R22 pad 1: /BM1397-1/GND1 -> Net-(U11-NRSTO)
- R22 pad 2: Net-(IC2-ADDR1) -> Net-(U14-NRSTI)
- R23 pad 1: /BM1397-1/GND1 -> Net-(U11-CO)
- R23 pad 2: Net-(IC2-ADDR2) -> Net-(U14-CI)
- R24 pad 1: Net-(U9-DN) -> /VDD
- R24 pad 2: /TEMP1_N -> /BM1366-1/GND
- R25 pad 1: Net-(U10-DN) -> /VDD
- R25 pad 2: /TEMP2_N -> /BM1366-1/GND
- R26 pad 1: /TEMP1_P -> Net-(U14-NRSTO)
- R26 pad 2: Net-(U9-DP) -> /BM1366-2/NRSTI
- R27 pad 1: /TEMP2_P -> Net-(U14-CO)
- R27 pad 2: Net-(U10-DP) -> /BM1366-2/CI
- R28 pad 1: /Fan/FAN_PWM1 -> Net-(U14-NC)
- R28 pad 2: /3V3 -> Net-(U14-MODE_1)
- R29 pad 1: /Fan/FAN_PWM2 -> Net-(U14-BO)
- R29 pad 2: /3V3 -> /BM1366-1/BO
- R3 pad 2: Net-(U1-IN-) -> Net-(U3-IN-)
- R30 pad 1: /Fan/FAN_TACH1 -> Net-(U14-CLKO)
- R30 pad 2: /3V3 -> /BM1366-1/CLKO
- R31 pad 1: /Fan/FAN_TACH2 -> Net-(U14-RI)
- R31 pad 2: /3V3 -> /BM1366-2/RO
- R32 pad 1: /BM1397-3/VDD3 -> /Fan/FAN_PWM1
- R32 pad 2: Net-(IC3-ADDR0) -> /3V3
- R33 pad 1: /BM1397-3/VDD3 -> /Fan/FAN1_TACH
- R33 pad 2: Net-(IC3-ADDR1) -> /3V3
- R34 pad 1: /BM1397-3/VDD3 -> /Fan/FAN2_TACH
- R34 pad 2: Net-(IC3-ADDR2) -> /3V3
- R35 pad 1: /BM1397-1/GND1 -> /BM1366-2/GND
- R35 pad 2: /BM1397-3/VDD3 -> Net-(U21-BI)
- R36 pad 1: /BM1397-1/GND1 -> Net-(U21-NC)
- R36 pad 2: /BM1397-3/VDD3 -> Net-(U21-MODE_1)
- R37 pad 1: /BM1397-3/VDD3 -> Net-(C86-Pad2)
- R38 pad 1: /BM1397-3/VDD3 -> /BM1366-1/GND
- R38 pad 2: Net-(IC4-ADDR1) -> /BM1366-2/GND
- R39 pad 1: /BM1397-3/VDD3 -> Net-(U21-RI)
- R4 pad 1: Net-(C8-Pad2) -> Net-(C9-Pad2)
- R40 pad 1: GND -> /BM1366-1/GND
- R40 pad 2: Net-(IC5-ADDR0) -> /BM1366-2/GND
- R41 pad 1: GND -> Net-(U21-BO)
- R42 pad 1: GND -> Net-(U21-CLKO)
- R45 pad 1: GND -> Net-(U22-NRSTO)
- R45 pad 2: Net-(IC6-ADDR0) -> /BM1366-3/NRSTI
- R46 pad 1: GND -> Net-(U22-CO)
- R46 pad 2: Net-(IC6-ADDR1) -> /BM1366-3/CI
- R47 pad 1: GND -> Net-(U22-NC)
- R47 pad 2: Net-(IC6-ADDR2) -> Net-(U22-MODE_1)
- R48 pad 1: Net-(U15-DN) -> Net-(U22-BO)
- R48 pad 2: /TEMP3_N -> /BM1366-2/BO
- R49 pad 1: /TEMP3_P -> Net-(U22-CLKO)
- R49 pad 2: Net-(U15-DP) -> /BM1366-2/CLKO
- R5 pad 1: /3V3 -> /Power/PGOOD
- R5 pad 2: /Power/PGOOD -> Net-(U4-BP)
- R50 pad 1: /Fan/FAN_PWM3 -> Net-(U22-RI)
- R50 pad 2: /3V3 -> /BM1366-3/RO
- R51 pad 1: /Fan/FAN_TACH3 -> GND
- R51 pad 2: /3V3 -> Net-(U25-BI)
- R6 pad 1: /Power/PGOOD -> Net-(Q2-G)
- R6 pad 2: Net-(U2-BP) -> GND
- R7 pad 1: Net-(Q2-G) -> /3V3
- R7 pad 2: GND -> /Power/PGOOD
- R8 pad 1: Net-(U5-FS0) -> /VDD
- R8 pad 2: GND -> Net-(C17-Pad1)
- R9 pad 2: Net-(C17-Pad1) -> /Power/OUT0
- TP10 pad 1: /Fan/FAN_TACH1 -> /Fan/FAN2_TACH
- TP11 pad 1: /Fan/FAN_TACH2 -> /Fan/FAN1_PWM
- TP12 pad 1: /Fan/FAN_PWM1 -> /Fan/FAN2_PWM
- TP13 pad 1: /Fan/FAN_PWM2 -> /BM1366-2/1V2
- TP14 pad 1: /BM1398-2/1V8 -> /BM1366-2/0V8
- TP16 pad 1: /BM1398-2/0V8 -> /BM1366-3/0V8
- TP7 pad 1: Net-(IC1-CLKI) -> /BM1366-1/1V2
- TP8 pad 1: /1V8 -> /BM1366-1/0V8
- TP9 pad 1: /BM1397-1/0V8 -> /Fan/FAN1_TACH
- U1 pad 1: Net-(U1-IN+) -> /Power/VIN_M
- U1 pad 2: Net-(U1-IN-) -> GND
- U1 pad 3: GND -> /5V
- U10 pad 1: /3V3 -> /BM1366-1/1V2
- U10 pad 2: Net-(U10-DP) -> /BM1366-1/GND
- U10 pad 3: Net-(U10-DN) -> /BM1366-1/CLKI
- U10 pad 4: /Fan/FAN_PWM2 -> /BM1366-1/1V2
- U11 pad 1: /5V -> Net-(U11-VDD1_0)
- U11 pad 2: /BM1397-3/VDD3 -> Net-(U11-VDD2_0)
- U11 pad 3: /5V -> Net-(U11-VDD3_0)
- U11 pad 4: unconnected-(U11-PG-Pad4) -> Net-(C32-Pad1)
- U11 pad 5: /BM1398-2/1V8 -> /NRSTI
- U12 pad 2: /BM1397-3/VDD3 -> /BM1366-1/GND
- U12 pad 5: /BM1398-2/0V8 -> /BM1366-1/1V2
- U13 pad 2: GND -> /BM1366-1/GND
- U13 pad 5: /BM1397-3/1V8 -> /BM1366-1/0V8
- U14 pad 1: /5V -> Net-(U11-VDD1_1)
- U14 pad 2: GND -> Net-(U11-VDD2_1)
- U14 pad 3: /5V -> Net-(U11-VDD3_1)
- U14 pad 4: unconnected-(U14-PG-Pad4) -> Net-(C48-Pad2)
- U14 pad 5: /BM1397-3/0V8 -> Net-(U14-NRSTI)
- U15 pad 1: /3V3 -> /SCL
- U15 pad 2: Net-(U15-DP) -> GND
- U15 pad 3: Net-(U15-DN) -> unconnected-(U15-ALERT-Pad3)
- U15 pad 4: /Fan/FAN_PWM3 -> unconnected-(U15-A0-Pad4)
- U15 pad 5: GND -> /3V3
- U15 pad 6: /Fan/FAN_TACH3 -> /SDA
- U16 pad 1: /1V8 -> /SCL
- U16 pad 3: /NRSTI -> unconnected-(U16-ALERT-Pad3)
- U16 pad 4: /NRSTI -> unconnected-(U16-A0-Pad4)
- U16 pad 5: GND -> /3V3
- U16 pad 6: /3V3 -> /SDA
- U17 pad 1: /1V8 -> /SDA
- U17 pad 2: GND -> /SCL
- U17 pad 3: /RO -> /3V3
- U17 pad 4: /RO -> GND
- U17 pad 5: /1V8 -> /Fan/FAN1_PWM
- U17 pad 6: /3V3 -> /Fan/FAN1_TACH
- U18 pad 1: /1V8 -> /3V3
- U18 pad 2: GND -> unconnected-(U18-DP-Pad2)
- U18 pad 3: /CI -> unconnected-(U18-DN-Pad3)
- U18 pad 4: /CI -> /Fan/FAN_PWM1
- U18 pad 6: /3V3 -> /Fan/FAN_TACH1
- U2 pad 1: /Power/VIN_M -> /5V
- U2 pad 2: Net-(U2-SS) -> GND
- U2 pad 3: /Power/PGOOD -> /5V
- U2 pad 4: Net-(U2-COMP) -> (no net)
- U2 pad 5: /Power/OUT0 -> /3V3
- U3 pad 1: /Power/VIN_M -> Net-(U3-IN+)
- U3 pad 2: GND -> Net-(U3-IN-)
- U3 pad 3: /5V -> GND
- U4 pad 1: /5V -> /Power/VIN_M
- U4 pad 2: GND -> Net-(U4-SS)
- U4 pad 3: /5V -> /Power/PGOOD
- U4 pad 4: (no net) -> Net-(U4-COMP)
- U4 pad 5: /3V3 -> /Power/OUT0
- U6 pad 1: GND -> /1V8
- U6 pad 2: /3V3 -> GND
- U6 pad 3: /ESP32/EN -> /NRSTI
- U6 pad 4: unconnected-(U6-GPIO4/TOUCH4/ADC1_CH3-Pad4) -> /NRSTI
- U6 pad 5: unconnected-(U6-GPIO5/TOUCH5/ADC1_CH4-Pad5) -> GND
- U6 pad 6: unconnected-(U6-GPIO6/TOUCH6/ADC1_CH5-Pad6) -> /3V3
- U7 pad 1: /5V -> /1V8
- U7 pad 2: /BM1397-1/GND1 -> GND
- U7 pad 3: /5V -> /RO
- U7 pad 4: unconnected-(U7-PG-Pad4) -> /RO
- U8 pad 1: /5V -> /1V8
- U8 pad 2: /BM1397-1/GND1 -> GND
- U8 pad 3: /5V -> /CI
- U8 pad 4: unconnected-(U8-PG-Pad4) -> /CI
- U8 pad 5: /BM1397-1/0V8 -> GND
- U9 pad 1: /3V3 -> GND
- U9 pad 2: Net-(U9-DP) -> /3V3
- U9 pad 3: Net-(U9-DN) -> /ESP32/EN
- U9 pad 4: /Fan/FAN_PWM1 -> unconnected-(U9-GPIO4/TOUCH4/ADC1_CH3-Pad4)
- U9 pad 5: GND -> unconnected-(U9-GPIO5/TOUCH5/ADC1_CH4-Pad5)
- U9 pad 6: /Fan/FAN_TACH1 -> unconnected-(U9-GPIO6/TOUCH6/ADC1_CH5-Pad6)
- U9 pad 7: /SDA -> unconnected-(U9-GPIO7/TOUCH7/ADC1_CH6-Pad7)
- U9 pad 8: /SCL -> /ESP32/XIN32
- USB1 pad 2: Net-(U6-GPIO19/U1RTS/ADC2_CH8/CLK_OUT2/USB_D-) -> Net-(U9-GPIO19/U1RTS/ADC2_CH8/CLK_OUT2/USB_D-)
- USB1 pad 3: Net-(U6-GPIO20/U1CTS/ADC2_CH9/CLK_OUT1/USB_D+) -> Net-(U9-GPIO20/U1CTS/ADC2_CH9/CLK_OUT1/USB_D+)
Routing:
- added copper zone on B.Cu, net /BM1366-1/GND
- added copper zone on F.Cu, net /BM1366-1/GND
- added copper zone on B.Cu, net GND
- removed copper zone on B.Cu, net /BM1397-1/GND1
- removed copper zone on F.Cu, net /BM1397-1/GND1
- removed copper zone on B.Cu, net /BM1397-3/VDD3
- removed copper zone on F.Cu, net /BM1397-3/VDD3

Commit message: very rough sorting and placement
Parts:
- moved C64 311.7 mm to (235.5, 80.5)
- moved D1 279.4 mm to (192.6, 26.3)
- moved C65 278.4 mm to (217.9, 77.1)
- moved U15 268.9 mm to (200.2, 76.7)
- moved C22 266.7 mm to (199.4, 38.7)
- moved R34 266.1 mm to (205.3, 72.3)
- moved R33 265.3 mm to (207.2, 77.0)
- moved C28 263.6 mm to (204.9, 33.4)
- moved R32 262.7 mm to (199.2, 62.9)
- moved C24 262.1 mm to (199.0, 33.4)
- moved C23 258.1 mm to (199.3, 28.9)
- moved J4 257.0 mm to (185.8, 77.1)
- moved R15 255.4 mm to (203.0, 36.2)
- moved R14 254.9 mm to (201.0, 36.2)
- moved R13 254.3 mm to (199.0, 36.2)
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Routing:
- net /BM1366-1/1V2: track 0.00 -> 6.16 mm
- net Net-(U11-VDD3_0): track 0.00 -> 1.82 mm
- net Net-(U11-NRSTO): track 0.00 -> 1.81 mm
Other:
- board text removed: "/ 21M"
- board text removed: "1V8"
- board text removed: "∞"

Commit message: more rough layout work
Parts:
- C69, C70: moved to F.Cu
- moved TP10 346.4 mm to (250.5, 47.9)
- moved TP9 345.0 mm to (250.5, 44.4)
- moved TP11 341.0 mm to (250.5, 51.5)
- moved TP12 341.0 mm to (250.5, 55.0)
- moved TP16 252.2 mm to (158.9, 154.6)
- moved TP13 216.2 mm to (115.6, 147.5)
- moved TP14 205.1 mm to (114.0, 162.8)
- moved TP8 169.9 mm to (76.0, 145.4)
- moved J6 168.5 mm to (246.7, 53.9)
- moved TP7 162.8 mm to (67.0, 157.7)
- moved C61 155.8 mm to (238.4, 58.9)
- moved C62 155.8 mm to (238.4, 60.9)
- moved C63 155.8 mm to (238.4, 62.9)
- moved R54 143.3 mm to (171.4, 141.4)
- moved R56 143.3 mm to (171.4, 146.3)
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Routing:
- net Net-(U11-VDD3_0): track 1.82 -> 10.3 mm
- net Net-(C32-Pad1): track 0.00 -> 8.29 mm
- net Net-(U11-VDD1_0): track 0.00 -> 7.42 mm
- net Net-(U11-VDD2_0): track 0.00 -> 7.08 mm
- net /VDD: track 0.00 -> 6.76 mm
- net /BM1366-1/1V2: track 6.16 -> 0.00 mm
- net Net-(U11-NRSTO): track 1.81 -> 0.00 mm
- net GND: vias 0 -> 18
- added copper zone on F.Cu, net /BM1366-2/GND
- added copper zone on F.Cu, net /Power/VIN_M
- added copper zone on F.Cu, net /VDD
- removed copper zone on B.Cu, net /BM1366-1/GND
- removed copper zone on B.Cu, net GND

Commit message: cleanup
Parts:
- moved C83 78.3 mm to (191.0, 143.5)
- moved C85 77.4 mm to (191.0, 145.4)
- moved C87 76.5 mm to (191.0, 147.4)
- moved C80 75.3 mm to (191.0, 141.5)
- moved C88 38.6 mm to (186.7, 145.6)
- moved C111 34.9 mm to (159.0, 116.5)
- moved C127 32.3 mm to (180.0, 115.0)
- moved C125 32.1 mm to (180.0, 113.0)
- moved C121 25.0 mm to (164.0, 113.0)
- moved C114 13.7 mm to (159.0, 118.4)
- moved C102 10.6 mm to (159.0, 112.5)
- moved R42 10.2 mm to (127.3, 104.1)
- moved R44 10.2 mm to (125.0, 104.8)
- moved R41 10.2 mm to (127.5, 102.2)
- moved C104 8.67 mm to (159.0, 114.5)
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Routing:
- net Net-(U11-VDD3_0): track 10.3 -> 1.80 mm
- net Net-(C32-Pad1): track 8.29 -> 0.00 mm
- net /VDD: track 6.76 -> 0.00 mm
- net Net-(U11-VDD2_0): track 7.08 -> 1.01 mm
- net Net-(U11-VDD1_0): track 7.42 -> 2.26 mm

Commit message: flip center asic pads
Parts:
- moved C93 20.3 mm to (126.1, 82.0), turned to 90 degrees
- moved R44 20.2 mm to (128.2, 84.9), turned to 90 degrees
- moved C78 19.8 mm to (122.2, 82.0), turned to 90 degrees
- moved R42 19.5 mm to (124.2, 84.9), turned to 90 degrees
- moved C82 18.5 mm to (124.1, 82.0), turned to 90 degrees
- moved R43 18.3 mm to (126.2, 84.9), turned to 90 degrees
- moved R41 18.1 mm to (122.2, 84.9), turned to 90 degrees
- moved U21 17.6 mm to (130.6, 97.4)
- moved C69 17.6 mm to (118.2, 82.0), turned to 90 degrees
- moved U22 17.5 mm to (113.0, 97.1)
- moved R39 16.8 mm to (120.2, 84.9), turned to 90 degrees
- moved C71 16.4 mm to (120.2, 82.0), turned to 90 degrees
- moved R37 16.1 mm to (118.2, 84.9), turned to 90 degrees
- moved C92 8.00 mm to (124.4, 104.1)
- moved C94 7.87 mm to (125.8, 104.0)
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
Commit message: alignment
Parts:
- moved C27 116.5 mm to (137.7, 25.5)
- moved U7 103.7 mm to (133.9, 28.4)
- moved U8 102.6 mm to (133.9, 33.0)
- moved C24 62.5 mm to (137.3, 23.1)
- moved C25 62.5 mm to (139.3, 23.1)
- moved C26 62.5 mm to (141.2, 23.1)
- moved C28 62.5 mm to (143.2, 23.1)
- moved U6 59.9 mm to (133.9, 23.9)
- moved C29 54.6 mm to (137.7, 27.5)
- moved R35 1.28 mm to (143.5, 87.2)
- moved U22 0.16 mm to (113.0, 97.3)
- moved U21 0.13 mm to (130.6, 97.3)
Changed lines of the file:
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@@
   )
   (footprint "lcsc:SOT-23-6_L2.9-W1.6-P0.95-LS2.8-BR" (layer "F.Cu")
-    (at 59.76 103.95)
+    (at 133.905 33.02)
     (property "JLC Part" "Extended Part")
     (property "LCSC Part" "C7843")
@@
   )
   (footprint "Capacitor_SMD:C_0402_1005Metric" (layer "F.Cu")
-    (at 200.95 33.36 -90)
+    (at 139.26 23.12 -90)
     (descr "Capacitor SMD 0402 (1005 Metric), square (rectangular) end terminal, IPC_7351 nominal, (Body size source: IPC-SM-782 page 76, https://www.pcb-3d.com/wordpress/wp-content/uploads/ipc-sm-782a_amendment_1_and_2.pdf), generated with kicad-footprint-generator")
     (tags "capacitor")
@@
   )
   (footprint "bitaxe:BM1366" (layer "F.Cu")
-    (at 130.6 97.4 180)
+    (at 130.6 97.268 180)
     (property "Sheetfile" "bm1366-2.kicad_sch")
     (property "Sheetname" "BM1366-2")
@@
   )
   (footprint "lcsc:SOT-23-6_L2.9-W1.6-P0.95-LS2.8-BR" (layer "F.Cu")
-    (at 55.96 96.84)
+    (at 133.905 28.44)
     (property "JLC Part" "Extended Part")
     (property "LCSC Part" "C7843")
@@
   )
   (footprint "bitaxe:BM1366" (layer "F.Cu")
-    (at 113 97.108 180)
+    (at 113 97.268 180)
     (property "Sheetfile" "bm1366-2.kicad_sch")
     (property "Sheetname" "BM1366-2")
@@
   )
   (footprint "Capacitor_SMD:C_0402_1005Metric" (layer "F.Cu")
-    (at 202.92 33.36 90)
+    (at 141.23 23.12 90)
     (descr "Capacitor SMD 0402 (1005 Metric), square (rectangular) end terminal, IPC_7351 nominal, (Body size source: IPC-SM-782 page 76, https://www.pcb-3d.com/wordpress/wp-content/uploads/ipc-sm-782a_amendment_1_and_2.pdf), generated with kicad-footprint-generator")
     (tags "capacitor")
@@
   )
   (footprint "Capacitor_SMD:C_0402_1005Metric" (layer "F.Cu")
-    (at 204.89 33.36 -90)
+    (at 143.2 23.12 -90)
     (descr "Capacitor SMD 0402 (1005 Metric), square (rectangular) end terminal, IPC_7351 nominal, (Body size source: IPC-SM-782 page 76, https://www.pcb-3d.com/wordpress/wp-content/uploads/ipc-sm-782a_amendment_1_and_2.pdf), generated with kicad-footprint-generator")
     (tags "capacitor")
@@
   )
   (footprint "bitaxe:BM1366" (layer "F.Cu")
-    (at 87.257743 97.218)
+    (at 87.257743 97.268)
     (property "Sheetfile" "bm1366-1.kicad_sch")
     (property "Sheetname" "BM1366-1")
@@
   )
   (footprint "Resistor_SMD:R_0402_1005Metric" (layer "F.Cu")
-    (at 143.327 88.469)
+    (at 143.49 87.2)
     (descr "Resistor SMD 0402 (1005 Metric), square (rectangular) end terminal, IPC_7351 nominal, (Body size source: IPC-SM-782 page 72, https://www.pcb-3d.com/wordpress/wp-content/uploads/ipc-sm-782a_amendment_1_and_2.pdf), generated with kicad-footprint-generator")
     (tags "resistor")
@@
   )
   (footprint "Capacitor_SMD:C_0402_1005Metric" (layer "F.Cu")
-    (at 191.28 38.19)
+    (at 137.74 27.51)
     (descr "Capacitor SMD 0402 (1005 Metric), square (rectangular) end terminal, IPC_7351 nominal, (Body size source: IPC-SM-782 page 76, https://www.pcb-3d.com/wordpress/wp-content/uploads/ipc-sm-782a_amendment_1_and_2.pdf), generated with kicad-footprint-generator")
     (tags "capacitor")
@@
   )
   (footprint "Capacitor_SMD:C_0402_1005Metric" (layer "F.Cu")
-    (at 57.04 109.53)
+    (at 137.74 25.54)
     (descr "Capacitor SMD 0402 (1005 Metric), square (rectangular) end terminal, IPC_7351 nominal, (Body size source: IPC-SM-782 page 76, https://www.pcb-3d.com/wordpress/wp-content/uploads/ipc-sm-782a_amendment_1_and_2.pdf), generated with kicad-footprint-generator")
     (tags "capacitor")
@@
   )
   (footprint "Capacitor_SMD:C_0402_1005Metric" (layer "F.Cu")
-    (at 198.98 33.36 -90)
+    (at 137.29 23.12 -90)
     (descr "Capacitor SMD 0402 (1005 Metric), square (rectangular) end terminal, IPC_7351 nominal, (Body size source: IPC-SM-782 page 76, https://www.pcb-3d.com/wordpress/wp-content/uploads/ipc-sm-782a_amendment_1_and_2.pdf), generated with kicad-footprint-generator")
     (tags "capacitor")
@@
   )
   (footprint "bitaxe:BM1366" (layer "F.Cu")
-    (at 69.85 97.218)
+    (at 69.85 97.268)
     (property "Sheetfile" "bm1366-1.kicad_sch")
     (property "Sheetname" "BM1366-1")
@@
   )
   (footprint "lcsc:SOT-23-6_L2.9-W1.6-P0.95-LS2.8-BR" (layer "B.Cu")
-    (at 172.42 69.755 180)
+    (at 133.905 23.86 180)
     (property "JLC Part" "Extended Part")
     (property "LCSC Part" "C7843")
@@
     (polygon
       (pts
-        (xy 67.69 100.45)
-        (xy 72.021 100.5)
+        (xy 67.8 100.45)
+        (xy 72 100.5)
         (xy 71.986 105.187)
         (xy 85.169 105.397)
@@
         (xy 89.434 100.276)
         (xy 89.442036 105.337963)
-        (xy 111 105.5)
-        (xy 110.95 100.493)
+        (xy 110.8 105.5)
+        (xy 110.8 100.493)
         (xy 115 100.5)
         (xy 115 105.336896)
         (xy 128.401 105.484)
-        (xy 128.373 100.673)
-        (xy 132.694 100.676)
-        (xy 132.8 109.6)
-        (xy 67.445 109.75)
+        (xy 128.373 100.473)
+        (xy 132.6 100.476)
+        (xy 132.6 109.6)
+        (xy 67.8 109.6)
       )
     )
@@
       (pts
         (xy 85.16 88.49)
-        (xy 89.5 88.5)
-        (xy 89.42 93.91)
+        (xy 89.4 88.5)
+        (xy 89.4 94)
         (xy 85.14 93.94)
       )
@@
     (polygon
       (pts
-        (xy 67.75 88.38)
+        (xy 67.8 88.38)
         (xy 71.99 88.39)
         (xy 72 94.12)
-        (xy 67.72 94.15)
+        (xy 67.8 94)
       )
     )
