File: bitaxeUltraHex.kicad_pcb (KiCad board)
At the start: 4 copper layers, 136.3 x 79.7 mm, 263 parts, among them J1 Conn_01x01, J2 Conn_01x01, J3 Conn_01x04, J4 TC2030-IDC, J5 Conn_01x04, J6 Conn_01x04, Q1 NTMFS5C673NLT1G, Q2 CSD17577Q5A, Q3 NTMFS5C673NLT1G, Q4 CSD17577Q5A, SW1 GT-TC029B-H025-L1N, SW2 GT-TC029B-H025-L1N, U1 uA7805, U10 25MHz, U11 BM1366_mode1, U12 MCP1824T-1202E, U13 MCP1824T-0802E, U14 BM1366_mode1, U15 TMP1075, U16 TMP1075, U17 EMC2302, U18 EMC2101, U19 MCP1824T-1202E, U2 RT9080-33GJ5, U20 MCP1824T-0802E, U21 BM1366_mode1, U22 BM1366_mode1, U23 MCP1824T-1202E, U24 MCP1824T-0802E, U25 BM1366_mode1, U26 BM1366_mode1, U3 INA219AIDCNR, U4 TPS40305, U5 DS4432U+, U6 SN74LVC1T45DBVR, U7 SN74LVC1T45DBVR, U8 SN74LVC1T45DBVR, U9 ESP32-S3-WROOM-1, Y1 32.768kHz

Commit message: Replace reference voltage regulators with new one
Parts:
- added C129: 0.1uF, Capacitor_SMD:C_0402_1005Metric, F.Cu at (161.8, 186.0)
- added C130: 1uF, Capacitor_SMD:C_0402_1005Metric, F.Cu at (161.8, 188.0)
- added R75: 243K, Resistor_SMD:R_0402_1005Metric, F.Cu at (48.7, 154.8)
- added R76: 536K, Resistor_SMD:R_0402_1005Metric, F.Cu at (48.7, 156.8)
- added R77: 634K, Resistor_SMD:R_0402_1005Metric, F.Cu at (48.7, 158.8)
- added R78: 536K, Resistor_SMD:R_0402_1005Metric, F.Cu at (48.7, 160.7)
- added R79: 243K, Resistor_SMD:R_0402_1005Metric, F.Cu at (108.4, 185.3)
- added R80: 536K, Resistor_SMD:R_0402_1005Metric, F.Cu at (108.4, 187.3)
- added R81: 634K, Resistor_SMD:R_0402_1005Metric, F.Cu at (108.4, 189.3)
- added R82: 536K, Resistor_SMD:R_0402_1005Metric, F.Cu at (108.4, 191.3)
- added R83: 243K, Resistor_SMD:R_0402_1005Metric, F.Cu at (158.9, 182.1)
- added R84: 536K, Resistor_SMD:R_0402_1005Metric, F.Cu at (158.9, 184.1)
- added R85: 634K, Resistor_SMD:R_0402_1005Metric, F.Cu at (158.9, 186.0)
- added R86: 536K, Resistor_SMD:R_0402_1005Metric, F.Cu at (158.9, 188.0)
- C107: value 0.1uF -> 1uF
- U12, U19, U23: value MCP1824T-1202E -> TLV752; footprint Package_TO_SOT_SMD:SOT-23-5 -> Package_SON:WSON-10-1EP_2.5x2.5mm_P0.5mm_EP1.2x2mm
- moved TP1 131.8 mm to (24.3, 43.4)
- moved TP2 131.8 mm to (20.3, 53.3)
- moved TP3 131.8 mm to (22.9, 53.3)
- moved TP4 131.8 mm to (25.5, 53.4)
- moved TP5 131.8 mm to (21.9, 47.5)
- moved TP6 131.8 mm to (24.4, 29.0)
- moved U23 56.7 mm to (160.6, 192.7)
- moved U19 49.9 mm to (115.1, 193.4)
- moved C106 47.4 mm to (161.8, 182.1)
- moved C76 45.9 mm to (111.3, 189.2)
- moved C73 44.0 mm to (111.3, 185.3)
- moved TP15 43.3 mm to (165.0, 182.8)
- moved TP13 38.6 mm to (114.5, 186.1)
- moved C41 34.9 mm to (54.1, 162.6)
- moved C107 34.7 mm to (161.8, 184.0)
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Connections:
- C107 pad 1: /5V -> /BM1366-3/1V2
- C108 pad 2: /BM1366-2/GND -> /FGND1
- C112 pad 1: /BM1366-2/GND -> /FGND1
- C122 pad 2: /BM1366-2/GND -> /FGND1
- C123 pad 1: /BM1366-2/GND -> /FGND1
- C35 pad 2: /BM1366-1/GND -> /FGND2
- C37 pad 1: /BM1366-1/GND -> /FGND2
- C39 pad 2: /BM1366-1/GND -> /FGND2
- C40 pad 2: /BM1366-1/GND -> /FGND2
- C41 pad 2: /BM1366-1/GND -> /FGND2
- C46 pad 1: /BM1366-1/1V2 -> /BM1366-1/0V8
- C46 pad 2: /BM1366-1/GND -> /FGND2
- C47 pad 1: /BM1366-1/0V8 -> /BM1366-1/1V2
- C47 pad 2: /BM1366-1/GND -> /FGND2
- C53 pad 2: /BM1366-1/GND -> /FGND2
- C57 pad 2: /BM1366-1/GND -> /FGND2
- C71 pad 2: /BM1366-2/GND -> /FGND1
- C73 pad 2: /BM1366-2/GND -> /FGND1
- C74 pad 2: /BM1366-2/GND -> /FGND1
- C75 pad 2: /BM1366-1/GND -> /FGND2
- C76 pad 1: /BM1366-2/1V2 -> /BM1366-2/0V8
- C76 pad 2: /BM1366-2/GND -> /FGND1
- C77 pad 1: /BM1366-2/0V8 -> /BM1366-2/1V2
- C77 pad 2: /BM1366-2/GND -> /FGND1
- C78 pad 2: /BM1366-2/GND -> /FGND1
- C79 pad 1: /BM1366-1/GND -> /FGND2
- C80 pad 1: /BM1366-1/GND -> /FGND2
- C80 pad 2: /BM1366-2/GND -> /FGND1
- C83 pad 1: /BM1366-1/GND -> /FGND2
- C83 pad 2: /BM1366-2/GND -> /FGND1
- C85 pad 1: /BM1366-1/GND -> /FGND2
- C85 pad 2: /BM1366-2/GND -> /FGND1
- C87 pad 1: /BM1366-1/GND -> /FGND2
- C87 pad 2: /BM1366-2/GND -> /FGND1
- C88 pad 1: /BM1366-1/GND -> /FGND2
- C88 pad 2: /BM1366-2/GND -> /FGND1
- C93 pad 2: /BM1366-2/GND -> /FGND1
- C94 pad 2: /BM1366-1/GND -> /FGND2
- C95 pad 1: /BM1366-1/GND -> /FGND2
- C97 pad 2: /BM1366-2/GND -> /FGND1
- R16 pad 1: /BM1366-1/GND -> /FGND2
- R24 pad 2: /BM1366-1/GND -> /FGND2
- R25 pad 2: /BM1366-1/GND -> /FGND2
- R35 pad 1: /BM1366-2/GND -> /FGND1
- R38 pad 1: /BM1366-1/GND -> /FGND2
- R38 pad 2: /BM1366-2/GND -> /FGND1
- R40 pad 1: /BM1366-1/GND -> /FGND2
- R40 pad 2: /BM1366-2/GND -> /FGND1
- R54 pad 1: /BM1366-2/GND -> /FGND1
- R56 pad 1: /BM1366-2/GND -> /FGND1
- TP13 pad 1: /BM1366-2/1V2 -> /BM1366-2/0V8
- TP14 pad 1: /BM1366-2/0V8 -> /BM1366-2/1V2
- TP15 pad 1: /BM1366-3/1V2 -> /BM1366-3/0V8
- TP16 pad 1: /BM1366-3/0V8 -> /BM1366-3/1V2
- TP7 pad 1: /BM1366-1/1V2 -> /BM1366-1/0V8
- TP8 pad 1: /BM1366-1/0V8 -> /BM1366-1/1V2
- U10 pad 2: /BM1366-1/GND -> /FGND2
- U11 pad 30: /BM1366-1/GND -> /FGND2
- U12 pad 1: /5V -> Net-(U12A-FB1)
- U12 pad 2: /BM1366-1/GND -> /FGND2
- U12 pad 4: unconnected-(U12-PG-Pad4) -> /FGND2
- U12 pad 5: /BM1366-1/1V2 -> /5V
- U14 pad 30: /BM1366-1/GND -> /FGND2
- U19 pad 1: /5V -> Net-(U19A-FB1)
- U19 pad 2: /BM1366-2/GND -> /FGND1
- U19 pad 4: unconnected-(U19-PG-Pad4) -> /FGND1
- U19 pad 5: /BM1366-2/1V2 -> /5V
- U21 pad 29: /BM1366-1/GND -> /FGND2
- U21 pad 30: /BM1366-2/GND -> /FGND1
- U22 pad 29: /BM1366-1/GND -> /FGND2
- U22 pad 30: /BM1366-2/GND -> /FGND1
- U23 pad 1: /5V -> Net-(U23A-FB1)
- U23 pad 4: unconnected-(U23-PG-Pad4) -> GND
- U23 pad 5: /BM1366-3/1V2 -> /5V
- U25 pad 29: /BM1366-2/GND -> /FGND1
- U26 pad 29: /BM1366-2/GND -> /FGND1
Routing:
- added copper zone on F.Cu, net /FGND1
- added copper zone on F.Cu, net /FGND2
- removed copper zone on F.Cu, net /BM1366-1/GND
- removed copper zone on F.Cu, net /BM1366-2/GND
