File: bitaxeUltraHex.kicad_sch (KiCad schematic)
At the start: 20 parts, among them J1 Screw Terminal, J2 Conn_01x01

Commit message: BOM mostly completed
Other:
- title: bitaxeUltraHex -> bitaxeHex
- moved on the sheet: H2, H4
Changed lines of the file:
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@@
   (paper "A")
   (title_block
-    (title "bitaxeUltraHex")
+    (title "bitaxeHex")
     (date "2023-06-11")
-    (rev "1")
+    (rev "300")
   )
   (junction (at 90.805 80.01) (diameter 0) (color 0 0 0 0)
@@
     )
   )
-  (symbol (lib_id "Mechanical:MountingHole") (at 85.725 190.5 0) (unit 1)
+  (symbol (lib_id "Mechanical:MountingHole") (at 85.09 190.5 0) (unit 1)
     (in_bom no) (on_board yes) (dnp no) (fields_autoplaced)
-    (property "Reference" "H4" (at 88.265 189.2299 0)
-      (effects (font (size 1.27 1.27)) (justify left))
-    )
-    (property "Value" "MountingHole" (at 88.265 191.7699 0)
-      (effects (font (size 1.27 1.27)) (justify left))
-    )
-    (property "Footprint" "bitaxe:4mm_mounting" (at 85.725 190.5 0)
-      (effects (font (size 1.27 1.27)) hide)
-    )
-    (property "Datasheet" "~" (at 85.725 190.5 0)
+    (property "Reference" "H4" (at 87.63 189.2299 0)
+      (effects (font (size 1.27 1.27)) (justify left))
+    )
+    (property "Value" "MountingHole" (at 87.63 191.7699 0)
+      (effects (font (size 1.27 1.27)) (justify left))
+    )
+    (property "Footprint" "bitaxe:4mm_mounting" (at 85.09 190.5 0)
+      (effects (font (size 1.27 1.27)) hide)
+    )
+    (property "Datasheet" "~" (at 85.09 190.5 0)
       (effects (font (size 1.27 1.27)) hide)
     )
@@
     )
   )
-  (symbol (lib_id "Mechanical:MountingHole") (at 85.725 176.53 0) (unit 1)
+  (symbol (lib_id "Mechanical:MountingHole") (at 85.09 176.53 0) (unit 1)
     (in_bom no) (on_board yes) (dnp no) (fields_autoplaced)
-    (property "Reference" "H2" (at 88.265 175.2599 0)
-      (effects (font (size 1.27 1.27)) (justify left))
-    )
-    (property "Value" "MountingHole" (at 88.265 177.7999 0)
-      (effects (font (size 1.27 1.27)) (justify left))
-    )
-    (property "Footprint" "bitaxe:4mm_mounting" (at 85.725 176.53 0)
-      (effects (font (size 1.27 1.27)) hide)
-    )
-    (property "Datasheet" "~" (at 85.725 176.53 0)
-      (effects (font (size 1.27 1.27)) hide)
-    )
+    (property "Reference" "H2" (at 87.63 175.2599 0)
+      (effects (font (size 1.27 1.27)) (justify left))
+    )
+    (property "Value" "MountingHole" (at 87.63 177.7999 0)
+      (effects (font (size 1.27 1.27)) (justify left))
+    )
+    (property "Footprint" "bitaxe:4mm_mounting" (at 85.09 176.53 0)
+      (effects (font (size 1.27 1.27)) hide)
+    )
+    (property "Datasheet" "~" (at 85.09 176.53 0)
+      (effects (font (size 1.27 1.27)) hide)
+    )
